File: smart-light/hardware/due-load-switch.kicad_sch (KiCad schematic)
At the start: 7 parts, among them J1 Due D22-D53 header, LHS row, Q1 IRLB8721PbF

Commit message: story(issue-31): make the load a blinky-style LED, not a 5 V lamp
LA1 (a 5 V module, <= 1 A) becomes D2, the same 5 mm red LED blinky uses,
with R14 = 330 ohm in series on the PS3 rail under Q1:

    +5V_LOAD -> R14 330R -> D2 anode ; cathode -> Q1 drain

I = (5.0 - 2.0) / 330 = 9.1 mA. Q1's drain-source drop contributes 1.4 mV
and does not enter the sum. Polarity is verified from the exported netlist
(+5V_LOAD -> R14.1, R14.2 -> D2.1 anode, D2.2 cathode -> Q1.2 drain), which
is the only mechanical proof of it; ERC reports zero violations.

The switching topology, the gate network and the 12k default-OFF argument
are unchanged - that argument is about the gate, and the gate does not know
what is on the drain, which is exactly why it was worth settling on paper.

What did change is every number the old 1 A load justified. Q1, PS3, C1 and
the star ground stay sized for a 1 A ceiling so a real 5 V light can replace
D2 with no other change, but nothing may now quote 1 A as the current that
flows today. So, throughout sheets 1-3 and the README, one rule: 1 A means
the ceiling the switch is built to permit, 9 mA is what D2 draws, and each
place says which it means.

  - ground bounce (sheet 2) is now two rows: 300 mV at the ceiling, 2.7 mV
    with D2 fitted, with the sheet stating the star ground buys nothing
    measurable today and is drawn for the ceiling because grounds cannot be
    re-planned after the fact
  - supply sizing gains a "load actually fitted" row; PS3 is ~200x the
    supply D2 needs
  - the MOSFET box says outright that a 62 A part switching 9 mA is a
    placeholder holding a size open, and marks the IRF540 counter-argument
    as applying at the ceiling only

R14 is numbered after R1-R13 rather than renumbering four sheets. The LAMP
symbol is dropped from the library. Three sheets whose only diff was an
export timestamp are left untouched.

Co-Authored-By: Claude Opus 4.8 <noreply@anthropic.com>
Parts:
- added D2: LED, red, symbol smart-light:LED
- R14: renamed from LA1; value 5 V light, <= 1 A -> 330R; symbol smart-light:LAMP -> smart-light:R
Connections:
- net at Q1.2 (D): now also D2.2; no longer R14.2
- new net: D2.1, R14.2
Other:
- note added: "anode to +5V_LOAD cathode to Q1's drain"
