File: arduino-due/blinky/hardware/due-blinky.kicad_sch (KiCad schematic)
At the start: 4 parts, among them J1 2x5 1.27 mm, on board, J2 2x5 1.27 mm, 3.3 V capable

Commit message: story(issue-43): the electrical feedback path that proves the LED actually lit
The blinky commanded PB26 and assumed it worked. Nothing downstream of that
store ever reported back, so a broken jumper, a reversed LED, an open resistor
and a dead output driver all produced identical firmware behaviour.

This is the diagram for closing that loop, and nothing else -- no firmware, no
build wiring, no code.

Rung 3 of the verify ladder, as an NPN low-side conduction sense: D1's return
current develops a base drive across R2, Q1 saturates, and its collector --
held up by R3 -- is dragged to VCE(sat). Active low on PA15 / D24, which is
the polarity hal.mmio.LevelInput's active_low option already exists for, so it
costs no new HAL contract.

Rungs 1 and 2 are insufficient rather than merely weak: an open circuit leaves
the pad at the commanded level, so neither ODSR nor PDSR can see it. And no
passive tap on D1 can work at all -- the only informative node in its branch
reaches at most VOH - Vf <= 3.30 - 1.60 = 1.70 V, which is 0.61 V short of
VIH (0.7 x VDDIO = 2.31 V, table 45-2). That is arithmetic, not a component
choice: a 3.3 V rail cannot carry an LED's forward drop and a valid logic
swing at once, so gain is mandatory. Q1's collector swings 3.10 V of the rail,
clearing the forbidden band by 0.79 V low and 0.99 V high.

R1 moves 1k -> 560 ohm to pay back the ~0.7 V Q1's base-emitter junction takes:
1.16 mA nominal, 1.88 mA worst case, 63 % of PB26's -3 mA Group-2 ceiling.
330 ohm and 220 ohm are now both over it.

The observability paradox is decided rather than left open. D1 is the board's
only output, so a detected load fault would have been reported through the
failed load. D2 on PD1 / D26 gives that report a path sharing nothing with
D1/R1/R2/R3/Q1. It does not contradict the fault response policy's rejection
of a second indicator: that clause was aimed at an indicator asserting health,
and D2 asserts only fault -- every way it can fail lands on dark.

Every electr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
Parts:
- added D2: LED (green), symbol due-blinky:LED
- added Q1: 2N3904, symbol due-blinky:NPN
- added R2, R3: 10k, symbol due-blinky:R
- added R4: 1k, symbol due-blinky:R
- R1: value 1k -> 560
Connections:
- net GND: now also D2.2, Q1.3 (E), R2.2; no longer D1.2
- net VTref_3V3 renamed +3V3
- net +3V3: now also R3.1
- new net: D1.2, Q1.1 (B), R2.1
- new net: D2.1, R4.2
- new net PA15_D24: Q1.2 (C), R3.2
- new net PD1_D26: R4.1
Other:
- note added: "The load on PB26 / D22, its feedback path, and the fault lamp"
- note removed: "External LED on PB26 / D22 - the blink indicator"
- title: Arduino Due blinky - SWD wiring and external LED -> Arduino Due blinky - SWD, external LED, feedback path
- moved on the sheet: D1, R1

Commit message: hardware(issue-44): as-built — D1 moves to PD1/D26, D2 takes PB26/D22
The board was wired with the two LED jumpers on each other's pins. The
schematic is the source of truth, so it now matches the bench rather than
the bench being rewired to match it: both pins were already justified on
the sheet against the same three tests, so the swap is legal as drawn.

What the swap actually changes is a per-pin current ceiling, not a label.
PB26 is Group 2 (-3 mA); PD1 is Group 1 (-15 mA).

  - R1's 560 ohm is no longer forced. It was sized to hold D1 under two
    thirds of -3 mA, and "330/220 ohm are illegal" was a PB26 fact. On
    PD1, D1's worst case is 13 % of -15 mA. 560 ohm is retained -- it is
    what is built and what every corner figure derives from -- but the
    sheet now records that it is a choice rather than a limit.
  - The hard lower bound moved to R4: D2 sits at 47 % of PB26's -3 mA, so
    keep R4 >= 470 ohm. This is the case R4's sizing was written for --
    it was sized against the Group 2 rule regardless of the pin it landed
    on, precisely so a jumper could move without re-deriving the sheet.

src/main.zig has to follow the diagram or the board blinks the fault lamp
and leaves D1 dark: PIOB/ID_PIOB -> PIOD base 0x400E1400 / ID_PIOD 14, and
the LED mask 1 << 26 -> 1 << 1. Confirmed against ArduinoCore-sam's
variant.cpp (PIN 26 = { PIOD, PIO_PD1, ID_PIOD, ... }) and the CMSIS
header rather than from memory. Flash 244 B -> 240 B; .data/.bss still 0.

Two things the swap adds that are worth wiring from, not assuming:

  - The header run no longer reads load-sense-lamp in order. Position 2
    is the FAULT LAMP, position 4 the BLINK LED.
  - At reset PD1 is a PIO input with its pull-up on, so D1 sees ~18 uA
    before firmware runs: dark, and not blinking.

Verified: netlist confirms PD1_D26 -> R1 and PB26_D22 -> R4 with the sense
on PA15_D24 untouched; ERC unchanged at 11 violations, 0 errors; the sheet
diff is 10 lines, all text, no wire or symbol move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
Connections:
- net PB26_D22: now also R4.1; no longer R1.1
- net PD1_D26: now also R1.1; no longer R4.1
Other:
- note added: "The load on PD1 / D26, its feedback path, and the fault lamp on PB26 / D22"
- note removed: "The load on PB26 / D22, its feedback path, and the fault lamp"
